File: pcb/motor-hub.kicad_sch (KiCad schematic)
At the start: 25 parts, among them J10 Conn_ARM_SWD_TagConnect_TC203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, SW1 SW_Push, SW2 SW_Push, U7 STM32G431CBUx, U8 74HC595, Y1 16MHz

Commit message: Finish lipo shutdown
Parts:
- removed C28: 100n, Capacitor_SMD:C_0402_1005Metric, symbol Device:C
- removed R25: R_Photo, Resistor_SMD:R_1210_3225Metric, symbol Device:R_Photo
- added R25: 1k5, Resistor_SMD:R_0402_1005Metric, symbol Device:R
Connections:
- net +3V3: no longer R24.1
- net GND: now also R25.2
- net AMB renamed BSNS
- net BSNS: now also R25.1
- new net VDD: R24.1
Other:
- note removed: "Photoresistor"

Commit message: Finish routing
Parts:
- removed C29: 100n, Capacitor_SMD:C_0402_1005Metric, symbol Device:C
Connections:
- net A1: now also U7.44 (PB6); no longer U7.41 (PB3)
- net A3: now also J10.4 (SWCLK), U7.37 (PA14); no longer U7.43 (PB5)
- net A5: now also U7.4 (PC15); no longer U7.3 (PC14)
- net B1: now also U7.43 (PB5); no longer U7.4 (PC15)
- net B2: now also U7.41 (PB3); no longer U7.29 (PC6)
- net B4: now also U7.45 (PB7); no longer U7.34 (PA12)
- net B5: now also U7.3 (PC14); no longer U7.45 (PB7)
- net BSNS: now also U7.27 (PB14); no longer U7.28 (PB15)
- net CR1: now also U7.47 (PB9); no longer U7.17 (PB0)
- net CR2: now also U7.11 (PA3); no longer U7.18 (PB1)
- net CR3: now also U7.14 (PA6); no longer U7.38 (PA15)
- net CR4: now also U7.17 (PB0); no longer U7.47 (PB9)
- net CR5: now also U7.28 (PB15); no longer U7.15 (PA7)
- net EN1: now also U7.9 (PA1); no longer U7.8 (PA0)
- net EN2: now also U7.10 (PA2); no longer U7.9 (PA1)
- net EN3: now also U7.13 (PA5); no longer U7.10 (PA2)
- net EN4: now also U7.18 (PB1); no longer U7.11 (PA3)
- net EN5: now also U7.29 (PC6); no longer U7.14 (PA6)
- net IR1: now also U7.8 (PA0); no longer U7.12 (PA4)
- net IR2: now also U7.12 (PA4); no longer U7.13 (PA5)
- net IR3: now also U7.15 (PA7); no longer U7.16 (PC4)
- net IR4: now also U7.16 (PC4); no longer U7.19 (PB2)
- net IR5: now also U7.19 (PB2); no longer U7.24 (PB11)
- net PH5: now also U7.26 (PB13); no longer U7.22 (PB10)
- net RCLK: now also U7.24 (PB11); no longer U7.27 (PB14)
- net RDAT: now also U7.25 (PB12); no longer U7.26 (PB13)
- net RSV: now also U7.22 (PB10); no longer U7.25 (PB12)
- net SIG1: now also U7.34 (PA12); no longer U7.30 (PA8)
- net SIG2: now also U7.33 (PA11); no longer U7.31 (PA9)
- net SIG4: now also U7.31 (PA9); no longer U7.33 (PA11)
- net SIG5: now also U7.30 (PA8); no longer J10.4 (SWCLK), U7.37 (PA14)
- net SL5: now also U7.38 (PA15); no longer U7.44 (PB6)
Other:
- moved on the sheet: C55

Commit message: Add power switch
Parts:
- FB1: LCSC (none) -> C1017
Changed lines of the file:
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@@
+			)
+		)
+		(property "LCSC" "C1017"
+			(at 119.38 33.02 90)
+			(effects
+				(font
+					(size 1.27 1.27)
+				)
+				(hide yes)
 			)
 		)

Commit message: Finish for revision 2 production
Parts:
- added C1: 100u, Capacitor_SMD:C_Elec_8x6.2, symbol Device:C
- R24: value 10k -> 33k; LCSC C25744 -> C25779
- R25: value 1k5 -> 7k5; LCSC C25867 -> C25918
- R26, R55: value 10k -> 7k5; LCSC C25744 -> C25918
Connections:
- net A1: now also U7.43 (PB5); no longer U7.44 (PB6)
- net A5: now also U7.3 (PC14); no longer U7.4 (PC15)
- net B1: now also U7.44 (PB6); no longer U7.43 (PB5)
- net B5: now also U7.4 (PC15); no longer U7.3 (PC14)
- net GND: now also C1.2
- net SIG1: now also U7.33 (PA11); no longer U7.34 (PA12)
- net SIG2: now also U7.34 (PA12); no longer U7.33 (PA11)
- net VDD: now also C1.1
- net SIG5 renamed PWR
Other:
- removed sheet Servo5
- note added: "Bulk Cap"
- moved on the sheet: C18, C30, C31, C34, C35, C55, J10, R24, R25, R26, R55, SW1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
